Commit message: Fix diablo gazebo relative.

File: urdf/common.xacro (robot description, xacro)
@@ -48,4 +48,5 @@
             <xacro:if value="${type == 'continuous'}">
                 <axis xyz="${axis_xyz}"/>
+                <limit effort="${effort}" velocity="${velocity}"/>
             </xacro:if>
             <xacro:if value="${type == 'prismatic'}">

File: urdf/diablo.urdf.xacro (robot description, xacro)
@@ -2,6 +2,5 @@
 <robot xmlns:xacro="http://ros.org/wiki/xacro">
     <!-- Include predefined materials -->
-    <xacro:include filename="$(find diablo)/description/urdf/imu/imu.urdf.xacro"/>
-    <xacro:include filename="$(find diablo)/description/urdf/common.xacro"/>
+    <xacro:include filename="$(find diablo)/urdf/common.xacro"/>
     <!-- Base Link -->
     <xacro:create_link name="diablo_base_link" mass="11.639" ixx="0.071628" ixy="-5.9879E-09" ixz="-0.00097471"
@@ -10,7 +9,4 @@
                        scale_factor="1" vision_scales="0.1 0.1 0.1"
                        collision_scales="0.1 0.001 0.1"/>
-    <xacro:IMU connected_to="diablo_base_link" imu_name="base_imu"
-               mesh_file="package://robot_common/include/robot_common/utilities/urdf/imu.stl" xyz="0.00 0.00 0.00"
-               rpy="0.00 0.00 0.00"/>
     <!--    main link-->
     <xacro:create_link name="left_thigh_link" mass="0.10382" ixx="3.6972E-05" ixy="2.4106E-05" ixz="4.3699E-10"
@@ -49,5 +45,5 @@
     <xacro:macro name="chassis" params="fixed_wheel='false' fixed_leg='false' close_chain='false' use_gazebo='false'">
         <xacro:if value="${use_gazebo}">
-            <xacro:include filename="$(find diablo)/description/urdf/gazebo.xacro"/>
+            <xacro:include filename="$(find diablo)/urdf/gazebo.xacro"/>
             <xacro:diablo_trans fixed_wheel="${fixed_wheel}" fixed_leg="${fixed_leg}" close_chain="${close_chain}"/>
             <xacro:if value="${close_chain}">
@@ -64,15 +60,15 @@
         </xacro:if>
         <xacro:unless value="${fixed_leg}">
-            <xacro:create_joint name="left_hip_joint" type="continuous" parent="left_fake_thigh_link" child="left_thigh_link"
-                                origin_xyz="0 0 0"
+            <xacro:create_joint name="left_hip_joint" type="revolute" parent="left_fake_thigh_link" child="left_thigh_link"
+                                origin_xyz="0 0 0" lower="-3.14" upper="3.14" effort="27" velocity="26"
                                 origin_rpy="0 0 -2.8729" axis_xyz="0 0 1"/>
-            <xacro:create_joint name="left_knee_joint" type="continuous" parent="left_thigh_link" child="left_shank_link"
-                                origin_xyz="0.14 0 0"
+            <xacro:create_joint name="left_knee_joint" type="revolute" parent="left_thigh_link" child="left_shank_link"
+                                origin_xyz="0.14 0 0" lower="-3.14" upper="3.14" effort="27" velocity="26"
                                 origin_rpy="0 0 2.8729" axis_xyz="0 0 1"/>
-            <xacro:create_joint name="right_hip_joint" type="continuous" parent="right_fake_thigh_link" child="right_thigh_link"
-                                origin_xyz="0 0 0"
+            <xacro:create_joint name="right_hip_joint" type="revolute" parent="right_fake_thigh_link" child="right_thigh_link"
+                                origin_xyz="0 0 0" lower="-3.14" upper="3.14" effort="27" velocity="26"
                                 origin_rpy="0 0 -2.8729" axis_xyz="0 0 1"/>
-            <xacro:create_joint name="right_knee_joint" type="continuous" parent="right_thigh_link" child="right_shank_link"
-                                origin_xyz="0.14 0 0"
+            <xacro:create_joint name="right_knee_joint" type="revolute" parent="right_thigh_link" child="right_shank_link"
+                                origin_xyz="0.14 0 0" lower="-3.14" upper="3.14" effort="27" velocity="26"
                                 origin_rpy="0 0 2.8729" axis_xyz="0 0 1"/>
             <xacro:if value="${close_chain}">
@@ -119,13 +115,13 @@
         <xacro:unless value="${fixed_wheel}">
             <xacro:create_joint name="left_wheel_joint" type="continuous" parent="left_shank_link" child="left_wheel"
-                                origin_xyz="0.14 0 0.0537" origin_rpy="0 0 0.13433" axis_xyz="0 0 1"/>
+                                origin_xyz="0.14 0 0.0537" origin_rpy="0 0 0.13433" axis_xyz="0 0 1" effort="27" velocity="26"/>
             <xacro:create_joint name="right_wheel_joint" type="continuous" parent="right_shank_link" child="right_wheel"
-                                origin_xyz="0.14 0 -0.0537" origin_rpy="0 0 -3.0073" axis_xyz="0 0 1"/>
+                                origin_xyz="0.14 0 -0.0537" origin_rpy="0 0 -3.0073" axis_xyz="0 0 1" effort="27" velocity="26"/>
         </xacro:unless>
         <xacro:if value="${fixed_wheel}">
             <xacro:create_joint name="left_wheel_joint" type="fixed" parent="left_shank_link" child="left_wheel"
-                                origin_xyz="0.14 0 0.0537" origin_rpy="0 0 0.13433" axis_xyz="0 0 1"/>
+                                origin_xyz="0.14 0 0.0537" origin_rpy="0 0 0.13433" />
             <xacro:create_joint name="right_wheel_joint" type="fixed" parent="right_shank_link" child="right_wheel"
-                                origin_xyz="0.14 0 -0.0537" origin_rpy="0 0 -3.0073" axis_xyz="0 0 1"/>
+                                origin_xyz="0.14 0 -0.0537" origin_rpy="0 0 -3.0073"/>
         </xacro:if>
     </xacro:macro>

File: urdf/diablo.xacro (robot description, xacro)
@@ -6,8 +6,17 @@
     <xacro:arg name="fixed_wheel" default="false"/>
     <xacro:arg name="use_gazebo" default="true"/>
-    <xacro:arg name="close_chain" default="true"/>
+    <xacro:arg name="close_chain" default="false"/>
+    <xacro:arg name="use_simulation" default="true"/>
     <xacro:if value="$(arg load_chassis)">
-        <xacro:include filename="$(find diablo)/description/urdf/diablo.urdf.xacro"/>
+        <xacro:include filename="$(find diablo)/urdf/diablo.urdf.xacro"/>
         <xacro:chassis fixed_wheel="$(arg fixed_wheel)" fixed_leg="$(arg fixed_leg)"  close_chain="$(arg close_chain)" use_gazebo="$(arg use_gazebo)"  />
     </xacro:if>
+    <xacro:if value="$(arg use_simulation)">
+        <gazebo>
+            <plugin name="robot_ros_control" filename="librobot_hw_sim.so">
+                <robotNamespace>/</robotNamespace>
+                <robotSimType>robot_gazebo/RobotHWSim</robotSimType>
+            </plugin>
+        </gazebo>
+    </xacro:if>
 </robot>

File: urdf/diablo_gazebo.urdf (robot description, URDF)
Before this commit: robot robot, 12 links, 11 joints
Links:
- removed link left_fake_shank_link
- removed link right_fake_shank_link
- link base_imu: geometry visual mesh filename=package://diablo/urdf/imu/imu.stl scale=1 1 1
Joints:
- removed joint left_fake_knee_joint
- removed joint right_fake_knee_joint
- joint left_fake_hip_joint: axis 0 0 1 -> (none); type continuous -> fixed
- joint left_hip_joint: limit (none) -> lower=-3.14 upper=3.14 effort=27 velocity=26; type continuous -> revolute
- joint left_knee_joint: limit (none) -> lower=-3.14 upper=3.14 effort=27 velocity=26; type continuous -> revolute
- joint left_wheel_joint: limit (none) -> effort=27 velocity=26
- joint right_fake_hip_joint: axis 0 0 1 -> (none); type continuous -> fixed
- joint right_hip_joint: limit (none) -> lower=-3.14 upper=3.14 effort=27 velocity=26; type continuous -> revolute
- joint right_knee_joint: limit (none) -> lower=-3.14 upper=3.14 effort=27 velocity=26; type continuous -> revolute
- joint right_wheel_joint: limit (none) -> effort=27 velocity=26

File: urdf/gazebo.xacro (robot description, xacro)
@@ -1,5 +1,9 @@
 <?xml version="1.0"?>
 <robot xmlns:xacro="http://ros.org/wiki/xacro" name="gazebo">
-    <xacro:include filename="$(find diablo)/description/urdf/common.xacro"/>
+    <xacro:include filename="$(find diablo)/urdf/common.xacro"/>
+    <xacro:include filename="$(find diablo)/urdf/imu/imu.urdf.xacro"/>
+    <xacro:IMU connected_to="diablo_base_link" imu_name="base_imu"
+               mesh_file="package://diablo/urdf/imu/imu.stl" xyz="0.00 0.00 0.00"
+               rpy="0.00 0.00 0.00"/>
     <xacro:macro name="diablo_trans" params="fixed_wheel='false' fixed_leg='false' close_chain='false'">
         <xacro:unless value="${fixed_leg}">
@@ -11,6 +15,8 @@
         </xacro:unless>
         <xacro:unless value="${fixed_wheel}">
-            <xacro:create_transmission joint_name="left_wheel_joint" hardware_interface="VelocityJointInterface"/>
-            <xacro:create_transmission joint_name="right_wheel_joint" hardware_interface="VelocityJointInterface"/>
+            <xacro:create_transmission joint_name="left_wheel_joint"/>
+            <xacro:create_transmission joint_name="right_wheel_joint"/>
+<!--            <xacro:create_transmission joint_name="left_wheel_joint" hardware_interface="VelocityJointInterface"/>-->
+<!--            <xacro:create_transmission joint_name="right_wheel_joint" hardware_interface="VelocityJointInterface"/>-->
         </xacro:unless>
         <xacro:if value="${close_chain}">
