Commit message: Could train move.

File: urdf/diablo_issac_gym.urdf (robot description, URDF)
Before this commit: robot robot, 10 links, 9 joints
Links:
- removed link base_imu
- link diablo_base_link: geometry collision mesh filename=../meshes/base_link.stl scale=0.1 0.001 0.1; visual mesh filename=../meshes/base_link.stl scale=0.1 0.1 0.1
- link left_fake_thigh_link: geometry collision mesh filename=../meshes/left_motor.STL scale=1 1 1; visual mesh filename=../meshes/left_motor.STL scale=1 1 1
- link left_shank_link: geometry collision mesh filename=../meshes/left_leg2.STL scale=1 1 1; visual mesh filename=../meshes/left_leg2.STL scale=1 1 1
- link left_thigh_link: geometry collision mesh filename=../meshes/left_leg1.STL scale=1 1 1; visual mesh filename=../meshes/left_leg1.STL scale=1 1 1
- link left_wheel: geometry collision mesh filename=../meshes/left_wheel.STL scale=1 1 1; visual mesh filename=../meshes/left_wheel.STL scale=1 1 1
- link right_fake_thigh_link: geometry collision mesh filename=../meshes/right_motor.STL scale=1 1 1; visual mesh filename=../meshes/right_motor.STL scale=1 1 1
- link right_shank_link: geometry collision mesh filename=../meshes/right_leg2.STL scale=1 1 1; visual mesh filename=../meshes/right_leg2.STL scale=1 1 1
- link right_thigh_link: geometry collision mesh filename=../meshes/right_leg1.STL scale=1 1 1; visual mesh filename=../meshes/right_leg1.STL scale=1 1 1
- link right_wheel: geometry collision mesh filename=../meshes/right_wheel.STL scale=1 1 1; visual mesh filename=../meshes/right_wheel.STL scale=1 1 1
Joints:
- removed joint base_imu_joint
- joint left_hip_joint: limit (none) -> lower=-3.14 upper=3.14 effort=100 velocity=1000; type continuous -> revolute
- joint left_knee_joint: limit (none) -> lower=-3.14 upper=3.14 effort=100 velocity=1000; type continuous -> revolute
- joint left_wheel_joint: limit (none) -> effort=5 velocity=1000; type continuous -> revolute
- joint right_hip_joint: limit (none) -> lower=-3.14 upper=3.14 effort=100 velocity=1000; type continuous -> revolute
- joint right_knee_joint: limit (none) -> lower=-3.14 upper=3.14 effort=100 velocity=1000; type continuous -> revolute
- joint right_wheel_joint: limit (none) -> effort=5 velocity=1000; type continuous -> revolute

Commit message: Add model and real motor config.

File: urdf/diablo_issac_gym.urdf (robot description, URDF)
Before this commit: robot robot, 9 links, 8 joints
Joints:
- joint left_hip_joint: limit lower=-3.14 upper=3.14 effort=100 velocity=1000 -> lower=-3.14 upper=3.14 effort=27 velocity=26
- joint left_knee_joint: limit lower=-3.14 upper=3.14 effort=100 velocity=1000 -> lower=-3.14 upper=3.14 effort=27 velocity=26
- joint left_wheel_joint: limit effort=5 velocity=1000 -> effort=27 velocity=1000
- joint right_hip_joint: limit lower=-3.14 upper=3.14 effort=100 velocity=1000 -> lower=-3.14 upper=3.14 effort=27 velocity=26
- joint right_knee_joint: limit lower=-3.14 upper=3.14 effort=100 velocity=1000 -> lower=-3.14 upper=3.14 effort=27 velocity=26
- joint right_wheel_joint: limit effort=5 velocity=1000 -> effort=27 velocity=26

Commit message: New train pt.

File: urdf/diablo_issac_gym.urdf (robot description, URDF)
Before this commit: robot robot, 9 links, 8 joints
Links:
- link diablo_base_link: geometry collision mesh filename=../meshes/base_link.stl scale=0.1 0.1 0.1; visual mesh filename=../meshes/base_link.stl scale=0.1 0.1 0.1
Joints:
- joint left_wheel_joint: limit effort=27 velocity=1000 -> effort=27 velocity=26

Commit message: Change mode.

File: urdf/diablo_issac_gym.urdf (robot description, URDF)
Before this commit: robot robot, 9 links, 8 joints
Links:
- link left_wheel: geometry collision cylinder length=0.05 radius=0.1; visual mesh filename=../meshes/left_wheel.STL scale=1 1 1
- link right_wheel: geometry collision cylinder length=0.05 radius=0.1; visual mesh filename=../meshes/left_wheel.STL scale=1 1 1

Commit message: New pt.

File: urdf/diablo_issac_gym.urdf (robot description, URDF)
Before this commit: robot robot, 9 links, 8 joints
Joints:
- joint left_hip_joint: limit lower=-3.14 upper=3.14 effort=27 velocity=26 -> lower=0.0 upper=2 effort=27 velocity=26
- joint left_knee_joint: limit lower=-3.14 upper=3.14 effort=27 velocity=26 -> lower=-1.5 upper=0.0 effort=27 velocity=26
- joint right_hip_joint: limit lower=-3.14 upper=3.14 effort=27 velocity=26 -> lower=0.0 upper=2 effort=27 velocity=26
- joint right_knee_joint: limit lower=-3.14 upper=3.14 effort=27 velocity=26 -> lower=-1.5 upper=0.0 effort=27 velocity=26

Commit message: Try diablo vmc as the same of gym.

File: urdf/diablo_issac_gym.urdf (robot description, URDF)
Before this commit: robot robot, 9 links, 8 joints
Joints:
- joint left_hip_joint: limit lower=0.0 upper=2 effort=27 velocity=26 -> lower=-1.57 upper=2 effort=27 velocity=26
- joint left_knee_joint: limit lower=-1.5 upper=0.0 effort=27 velocity=26 -> lower=-2 upper=0.0 effort=27 velocity=26
- joint right_hip_joint: limit lower=0.0 upper=2 effort=27 velocity=26 -> lower=-1.57 upper=2 effort=27 velocity=26
- joint right_knee_joint: limit lower=-1.5 upper=0.0 effort=27 velocity=26 -> lower=-2 upper=0.0 effort=27 velocity=26

Commit message: New pt.

File: urdf/diablo_issac_gym.urdf (robot description, URDF)
Before this commit: robot robot, 9 links, 8 joints
Joints:
- joint left_hip_joint: limit lower=-1.57 upper=2 effort=27 velocity=26 -> lower=0 upper=2 effort=27 velocity=26
- joint right_hip_joint: limit lower=-1.57 upper=2 effort=27 velocity=26 -> lower=0 upper=2 effort=27 velocity=26
