Commit message: Change wheel collision to cylinder.

File: urdf/diablo.urdf.xacro (robot description, xacro)
@@ -18,8 +18,23 @@
                        mesh_file="package://diablo/meshes/left_leg2.STL"
                        scale_factor="1"/>
-    <xacro:create_link name="left_wheel" mass="2.9494" ixx="0.0069338" ixy="2.8693E-09" ixz="4.6779E-09" iyy="0.006934"
-                       iyz="-5.0441E-11" izz="0.012567"
-                       mesh_file="package://diablo/meshes/left_wheel.STL"
-                       scale_factor="1"/>
+    <link name="left_wheel">
+        <inertial>
+            <origin rpy="0 0 0" xyz="0 0 0"/>
+            <mass value="2.9494"/>
+            <inertia ixx="0.0069338" ixy="2.8693e-09" ixz="4.6779e-09" iyy="0.006934" iyz="-5.0441e-11" izz="0.012567"/>
+        </inertial>
+        <visual>
+            <origin rpy="0 0 0" xyz="0 0 0"/>
+            <geometry>
+                <cylinder radius="0.1" length="0.05"/>
+            </geometry>
+        </visual>
+        <collision>
+            <origin rpy="0 0 0" xyz="0 0 0"/>
+            <geometry>
+                <cylinder radius="0.1" length="0.05"/>
+            </geometry>
+        </collision>
+    </link>
     <xacro:create_link name="right_thigh_link" mass="0.10382" ixx="3.6972E-05" ixy="2.4106E-05" ixz="-4.3686E-10"
                        iyy="0.00029278" iyz="4.1459E-11" izz="0.00032532"
@@ -30,8 +45,23 @@
                        mesh_file="package://diablo/meshes/right_leg2.STL"
                        scale_factor="1"/>
-    <xacro:create_link name="right_wheel" mass="2.9494" ixx="0.0069339" ixy="-1.3146E-07" ixz="-3.0392E-09"
-                       iyy="0.0069339" iyz="-3.5756E-09" izz="0.012567"
-                       mesh_file="package://diablo/meshes/right_wheel.STL"
-                       scale_factor="1"/>
+    <link name="right_wheel">
+        <inertial>
+            <origin rpy="0 0 0" xyz="0 0 0"/>
+            <mass value="2.9494"/>
+            <inertia ixx="0.0069339" ixy="-1.3146e-07" ixz="-3.0392e-09" iyy="0.0069339" iyz="-3.5756e-09" izz="0.012567"/>
+        </inertial>
+        <visual>
+            <origin rpy="0 0 0" xyz="0 0 0"/>
+            <geometry>
+                <cylinder radius="0.1" length="0.05"/>
+            </geometry>
+        </visual>
+        <collision>
+            <origin rpy="0 0 0" xyz="0 0 0"/>
+            <geometry>
+                <cylinder radius="0.1" length="0.05"/>
+            </geometry>
+        </collision>
+    </link>
     <!-- indispensable fake link-->
     <xacro:create_link name="left_fake_thigh_link" mass="1.3837" ixx="0.003352" ixy="2.7785E-09" ixz="-6.5913E-05" iyy="0.0034908"

File: urdf/diablo_issac_gym.urdf (robot description, URDF)
Before this commit: robot robot, 9 links, 8 joints
Links:
- link left_wheel: geometry collision cylinder length=0.05 radius=0.1; visual cylinder length=0.05 radius=0.1
- link right_wheel: geometry collision cylinder length=0.05 radius=0.1; visual cylinder length=0.05 radius=0.1

Commit message: Add vmc relative.

File: urdf/diablo.urdf.xacro (robot description, xacro)
@@ -9,4 +9,10 @@
                        scale_factor="1" vision_scales="0.1 0.1 0.1"
                        collision_scales="0.1 0.1 0.1"/>
+<!--    <link name="world"/>-->
+<!--    <joint name="world_to_base" type="fixed">-->
+<!--        <parent link="world"/>-->
+<!--        <child link="diablo_base_link"/>-->
+<!--        <origin xyz="0 0 0.3" rpy="0 0 0"/>-->
+<!--    </joint>-->
     <!--    main link-->
     <xacro:create_link name="left_thigh_link" mass="0.10382" ixx="3.6972E-05" ixy="2.4106E-05" ixz="4.3699E-10"
@@ -103,14 +109,14 @@
                                 origin_rpy="0 0 2.8729" axis_xyz="0 0 1"/>
             <xacro:if value="${close_chain}">
-                <xacro:create_joint name="left_fake_hip_joint" type="continuous" parent="diablo_base_link" child="left_fake_thigh_link"
-                                    origin_xyz="0 0.18755 0" origin_rpy="1.5708 0.13433 -3.1416" axis_xyz="0 0 1"/>
-                <xacro:create_joint name="left_fake_knee_joint" type="continuous" parent="left_fake_thigh_link" child="left_fake_shank_link"
+                <xacro:create_joint name="left_fake_hip_joint" type="revolute" parent="diablo_base_link" child="left_fake_thigh_link"
+                                    origin_xyz="0 0.18755 0" origin_rpy="1.5708 0.13433 -3.1416" axis_xyz="0 0 1" lower="-3.14" upper="3.14" effort="27" velocity="26"/>
+                <xacro:create_joint name="left_fake_knee_joint" type="revolute" parent="left_fake_thigh_link" child="left_fake_shank_link"
                                     origin_xyz="0.09 0 0"
-                                    origin_rpy="0 0 -2.8729" axis_xyz="0 0 1"/>
-                <xacro:create_joint name="right_fake_hip_joint" type="continuous" parent="diablo_base_link" child="right_fake_thigh_link"
-                                    origin_xyz="0 -0.18755 0" origin_rpy="1.5708 0.13433 3.1416" axis_xyz="0 0 1"/>
-                <xacro:create_joint name="right_fake_knee_joint" type="continuous" parent="right_fake_thigh_link" child="right_fake_shank_link"
+                                    origin_rpy="0 0 -2.8729" axis_xyz="0 0 1" lower="-3.14" upper="3.14" effort="27" velocity="26"/>
+                <xacro:create_joint name="right_fake_hip_joint" type="revolute" parent="diablo_base_link" child="right_fake_thigh_link"
+                                    origin_xyz="0 -0.18755 0" origin_rpy="1.5708 0.13433 3.1416" axis_xyz="0 0 1" lower="-3.14" upper="3.14" effort="27" velocity="26"/>
+                <xacro:create_joint name="right_fake_knee_joint" type="revolute" parent="right_fake_thigh_link" child="right_fake_shank_link"
                                     origin_xyz="0.09 0 0"
-                                    origin_rpy="0 0 -2.8729" axis_xyz="0 0 1"/>
+                                    origin_rpy="0 0 -2.8729" axis_xyz="0 0 1" lower="-3.14" upper="3.14" effort="27" velocity="26"/>
             </xacro:if>
             <xacro:unless value="${close_chain}">

File: urdf/diablo.xacro (robot description, xacro)
@@ -6,5 +6,5 @@
     <xacro:arg name="fixed_wheel" default="false"/>
     <xacro:arg name="use_gazebo" default="true"/>
-    <xacro:arg name="close_chain" default="false"/>
+    <xacro:arg name="close_chain" default="true"/>
     <xacro:arg name="use_simulation" default="true"/>
     <xacro:if value="$(arg load_chassis)">

Commit message: Change urdf.

File: urdf/diablo.urdf.xacro (robot description, xacro)
@@ -55,5 +55,5 @@
             <origin rpy="0 0 0" xyz="0 0 0"/>
             <mass value="2.9494"/>
-            <inertia ixx="0.0069339" ixy="-1.3146e-07" ixz="-3.0392e-09" iyy="0.0069339" iyz="-3.5756e-09" izz="0.012567"/>
+            <inertia ixx="0.0069338" ixy="2.8693e-09" ixz="4.6779e-09" iyy="0.006934" iyz="-5.0441e-11" izz="0.012567"/>
         </inertial>
         <visual>
@@ -153,5 +153,5 @@
                                 origin_xyz="0.14 0 0.0537" origin_rpy="0 0 0.13433" axis_xyz="0 0 1" lower="-1e10" upper="1e10" effort="27" velocity="26"/>
             <xacro:create_joint name="right_wheel_joint" type="revolute" parent="right_shank_link" child="right_wheel"
-                                origin_xyz="0.14 0 -0.0537" origin_rpy="0 0 -3.0073" axis_xyz="0 0 1" lower="-1e10" upper="1e10" effort="27" velocity="26"/>
+                                origin_xyz="0.14 0 -0.0537" origin_rpy="0 0 0.13433" axis_xyz="0 0 1" lower="-1e10" upper="1e10" effort="27" velocity="26"/>
         </xacro:unless>
         <xacro:if value="${fixed_wheel}">
@@ -159,5 +159,5 @@
                                 origin_xyz="0.14 0 0.0537" origin_rpy="0 0 0.13433" axis_xyz="0 0 1"/>
             <xacro:create_joint name="right_wheel_joint" type="fixed" parent="right_shank_link" child="right_wheel"
-                                origin_xyz="0.14 0 -0.0537" origin_rpy="0 0 -3.0073" axis_xyz="0 0 1"/>
+                                origin_xyz="0.14 0 -0.0537" origin_rpy="0 0 0.13433" axis_xyz="0 0 1"/>
         </xacro:if>
     </xacro:macro>

Commit message: Change urdf for real diablo.

File: urdf/diablo.urdf.xacro (robot description, xacro)
@@ -79,5 +79,5 @@
                        mesh_file="package://diablo/meshes/right_motor.STL"
                        scale_factor="1"/>
-    <xacro:macro name="chassis" params="fixed_wheel='false' fixed_leg='false' close_chain='false' use_gazebo='false'">
+    <xacro:macro name="chassis" params="fixed_wheel='false' fixed_leg='false' close_chain='false' use_gazebo='false' use_simulation='false'">
         <xacro:if value="${use_gazebo}">
             <xacro:include filename="$(find diablo)/urdf/gazebo.xacro"/>
@@ -110,19 +110,27 @@
             <xacro:if value="${close_chain}">
                 <xacro:create_joint name="left_fake_hip_joint" type="revolute" parent="diablo_base_link" child="left_fake_thigh_link"
-                                    origin_xyz="0 0.18755 0" origin_rpy="1.5708 0.13433 -3.1416" axis_xyz="0 0 1" lower="-1" upper="0.8" effort="27" velocity="26"/>
+                                    origin_xyz="0 0.18755 0" origin_rpy="1.5708 0.13433 -3.1416" axis_xyz="0 0 1" lower="-1.57" upper="1.57" effort="27" velocity="26"/>
                 <xacro:create_joint name="left_fake_knee_joint" type="revolute" parent="left_fake_thigh_link" child="left_fake_shank_link"
                                     origin_xyz="0.09 0 0"
-                                    origin_rpy="0 0 -2.8729" axis_xyz="0 0 1" lower="-0" upper="1.2" effort="27" velocity="26"/>
+                                    origin_rpy="0 0 -2.8729" axis_xyz="0 0 1" lower="-1.57" upper="1.57" effort="27" velocity="26"/>
                 <xacro:create_joint name="right_fake_hip_joint" type="revolute" parent="diablo_base_link" child="right_fake_thigh_link"
-                                    origin_xyz="0 -0.18755 0" origin_rpy="1.5708 0.13433 3.1416" axis_xyz="0 0 1" lower="-1" upper="0.8" effort="27" velocity="26"/>
+                                    origin_xyz="0 -0.18755 0" origin_rpy="1.5708 0.13433 3.1416" axis_xyz="0 0 1" lower="-1.57" upper="1.57" effort="27" velocity="26"/>
                 <xacro:create_joint name="right_fake_knee_joint" type="revolute" parent="right_fake_thigh_link" child="right_fake_shank_link"
                                     origin_xyz="0.09 0 0"
-                                    origin_rpy="0 0 -2.8729" axis_xyz="0 0 1" lower="-0" upper="1.2" effort="27" velocity="26"/>
+                                    origin_rpy="0 0 -2.8729" axis_xyz="0 0 1" lower="-1.57" upper="1.57" effort="27" velocity="26"/>
             </xacro:if>
             <xacro:unless value="${close_chain}">
-                <xacro:create_joint name="left_fake_hip_joint" type="fixed" parent="diablo_base_link" child="left_fake_thigh_link"
-                                    origin_xyz="0 0.18755 0" origin_rpy="1.5708 0.13433 -3.1416" axis_xyz="0 0 1"/>
-                <xacro:create_joint name="right_fake_hip_joint" type="fixed" parent="diablo_base_link" child="right_fake_thigh_link"
-                                    origin_xyz="0 -0.18755 0" origin_rpy="1.5708 0.13433 3.1416" axis_xyz="0 0 1"/>
+                <xacro:unless value="${use_simulation}">
+                    <xacro:create_joint name="left_fake_hip_joint" type="revolute" parent="diablo_base_link" child="left_fake_thigh_link"
+                                        origin_xyz="0 0.18755 0" origin_rpy="1.5708 0.13433 -3.1416" axis_xyz="0 0 1" lower="-1.57" upper="1.57" effort="27" velocity="26"/>
+                    <xacro:create_joint name="right_fake_hip_joint" type="revolute" parent="diablo_base_link" child="right_fake_thigh_link"
+                                        origin_xyz="0 -0.18755 0" origin_rpy="1.5708 0.13433 3.1416" axis_xyz="0 0 1" lower="-1.57" upper="1.57" effort="27" velocity="26"/>
+                </xacro:unless>
+                <xacro:if value="${use_simulation}">
+                    <xacro:create_joint name="left_fake_hip_joint" type="fixed" parent="diablo_base_link" child="left_fake_thigh_link"
+                                        origin_xyz="0 0.18755 0" origin_rpy="1.5708 0.13433 -3.1416" axis_xyz="0 0 1"/>
+                    <xacro:create_joint name="right_fake_hip_joint" type="fixed" parent="diablo_base_link" child="right_fake_thigh_link"
+                                        origin_xyz="0 -0.18755 0" origin_rpy="1.5708 0.13433 3.1416" axis_xyz="0 0 1"/>
+                </xacro:if>
             </xacro:unless>
         </xacro:unless>

File: urdf/diablo.xacro (robot description, xacro)
@@ -6,9 +6,9 @@
     <xacro:arg name="fixed_wheel" default="false"/>
     <xacro:arg name="use_gazebo" default="true"/>
-    <xacro:arg name="close_chain" default="true"/>
-    <xacro:arg name="use_simulation" default="true"/>
+    <xacro:arg name="close_chain" default="false"/>
+    <xacro:arg name="use_simulation" default="false"/>
     <xacro:if value="$(arg load_chassis)">
         <xacro:include filename="$(find diablo)/urdf/diablo.urdf.xacro"/>
-        <xacro:chassis fixed_wheel="$(arg fixed_wheel)" fixed_leg="$(arg fixed_leg)"  close_chain="$(arg close_chain)" use_gazebo="$(arg use_gazebo)"  />
+        <xacro:chassis fixed_wheel="$(arg fixed_wheel)" fixed_leg="$(arg fixed_leg)"  close_chain="$(arg close_chain)" use_gazebo="$(arg use_gazebo)" use_simulation="$(arg use_simulation)" />
     </xacro:if>
     <xacro:if value="$(arg use_simulation)">

Commit message: Fix inertial.

File: urdf/diablo.urdf.xacro (robot description, xacro)
@@ -4,5 +4,5 @@
     <xacro:include filename="$(find diablo)/urdf/common.xacro"/>
     <!-- Base Link -->
-    <xacro:create_link name="diablo_base_link" mass="11.639" ixx="0.071628" ixy="-5.9879E-09" ixz="-0.00097471"
+    <xacro:create_link name="diablo_base_link" mass="7" ixx="0.071628" ixy="-5.9879E-09" ixz="-0.00097471"
                        iyy="0.16274" iyz="-1.6369E-08" izz="0.14673"
                        mesh_file="package://diablo/meshes/base_link.stl"
@@ -71,10 +71,10 @@
     </link>
     <!-- indispensable fake link-->
-    <xacro:create_link name="left_fake_thigh_link" mass="1.3837" ixx="0.003352" ixy="2.7785E-09" ixz="-6.5913E-05" iyy="0.0034908"
-                       iyz="4.5045E-10" izz="0.0034856"
+    <xacro:create_link name="left_fake_thigh_link" mass="2.5" ixx="0.006704" ixy="5.557E-09" ixz="-0.000131826" iyy="0.0069816"
+                       iyz="9.009E-10" izz="0.0069712"
                        mesh_file="package://diablo/meshes/left_motor.STL"
                        scale_factor="1"/>
-    <xacro:create_link name="right_fake_thigh_link" mass="1.3838" ixx="0.003352" ixy="-2.6527E-09" ixz="6.5914E-05"
-                       iyy="0.0034908" iyz="-7.2968E-10" izz="0.0034856"
+    <xacro:create_link name="right_fake_thigh_link" mass="2.5" ixx="0.006704" ixy="-5.557E-09" ixz="0.000131826" iyy="0.0069816"
+                       iyz="-9.009E-10" izz="0.0069712"
                        mesh_file="package://diablo/meshes/right_motor.STL"
                        scale_factor="1"/>

File: urdf/diablo_ASM.urdf (robot description, URDF)
Before this commit: robot diablo_ASM, 7 links, 6 joints
Links:
- link diablo_base_link: mass 6 -> 7

File: urdf/diablo_ASM.xacro (robot description, xacro)
@@ -4,5 +4,5 @@
     <xacro:include filename="$(find diablo)/urdf/common.xacro"/>
     <!-- Base Link -->
-    <xacro:create_link name="diablo_base_link" mass="11.639" ixx="0.071628" ixy="-5.9879E-09" ixz="-0.00097471"
+    <xacro:create_link name="diablo_base_link" mass="7" ixx="0.071628" ixy="-5.9879E-09" ixz="-0.00097471"
                        iyy="0.16274" iyz="-1.6369E-08" izz="0.14673"
                        mesh_file="package://diablo/meshes/base_link.stl"
@@ -25,10 +25,10 @@
                        scale_factor="1"/>
     <!-- indispensable fake link-->
-    <xacro:create_link name="left_fake_thigh_link" mass="1.3837" ixx="0.003352" ixy="2.7785E-09" ixz="-6.5913E-05" iyy="0.0034908"
-                       iyz="4.5045E-10" izz="0.0034856"
+    <xacro:create_link name="left_fake_thigh_link" mass="2.5" ixx="0.006704" ixy="5.557E-09" ixz="-0.000131826" iyy="0.0069816"
+                       iyz="9.009E-10" izz="0.0069712"
                        mesh_file="package://diablo/meshes/left_motor.STL"
                        scale_factor="1"/>
-    <xacro:create_link name="right_fake_thigh_link" mass="1.3838" ixx="0.003352" ixy="-2.6527E-09" ixz="6.5914E-05"
-                       iyy="0.0034908" iyz="-7.2968E-10" izz="0.0034856"
+    <xacro:create_link name="right_fake_thigh_link" mass="2.5" ixx="0.006704" ixy="-5.557E-09" ixz="0.000131826" iyy="0.0069816"
+                       iyz="-9.009E-10" izz="0.0069712"
                        mesh_file="package://diablo/meshes/right_motor.STL"
                        scale_factor="1"/>
