Commit message: Fix ASM urdf.

File: urdf/diablo_ASM.urdf (robot description, URDF)
Before this commit: robot diablo_ASM, 7 links, 6 joints
Links:
- link diablo_base_link: geometry collision mesh filename=../meshes/base_link.stl scale=0.1 0.1 0.1; visual mesh filename=../meshes/base_link.stl scale=0.1 0.1 0.1
- link left_fake_shank_link: geometry collision mesh filename=../meshes/left_leg3.STL scale=1 1 1; visual mesh filename=../meshes/left_leg3.STL scale=1 1 1
- link left_fake_thigh_link: geometry collision mesh filename=../meshes/left_motor.STL scale=1 1 1; visual mesh filename=../meshes/left_motor.STL scale=1 1 1
- link left_wheel: geometry collision mesh filename=../meshes/left_wheel.STL scale=1 1 1; visual mesh filename=../meshes/left_wheel.STL scale=1 1 1
- link right_fake_shank_link: geometry collision mesh filename=../meshes/right_leg3.STL scale=1 1 1; visual mesh filename=../meshes/right_leg3.STL scale=1 1 1
- link right_fake_thigh_link: geometry collision mesh filename=../meshes/right_motor.STL scale=1 1 1; visual mesh filename=../meshes/right_motor.STL scale=1 1 1
- link right_wheel: geometry collision mesh filename=../meshes/right_wheel.STL scale=1 1 1; visual mesh filename=../meshes/right_wheel.STL scale=1 1 1
Joints:
- joint left_wheel_joint: origin xyz=0.14 0 0.0537 rpy=0 0 0.13433 -> xyz=0.14 0 0.025 rpy=0 0 0.13433
- joint right_wheel_joint: origin xyz=0.14 0 -0.0537 rpy=0 0 0.13433 -> xyz=0.14 0 -0.025 rpy=0 0 0.13433

File: urdf/diablo_ASM.xacro (robot description, xacro)
@@ -52,6 +52,6 @@
                         origin_rpy="0 0 -2.8729" axis_xyz="0 0 1" lower="-1.57" upper="1.57" effort="27" velocity="26"/>
     <xacro:create_joint name="left_wheel_joint" type="revolute" parent="left_fake_shank_link" child="left_wheel"
-                        origin_xyz="0.14 0 0.0537" origin_rpy="0 0 0.13433" axis_xyz="0 0 1" lower="-1e10" upper="1e10" effort="27" velocity="26"/>
+                        origin_xyz="0.14 0 0.025" origin_rpy="0 0 0.13433" axis_xyz="0 0 1" lower="-1e10" upper="1e10" effort="27" velocity="26"/>
     <xacro:create_joint name="right_wheel_joint" type="revolute" parent="right_fake_shank_link" child="right_wheel"
-                        origin_xyz="0.14 0 -0.0537" origin_rpy="0 0 0.13433" axis_xyz="0 0 1" lower="-1e10" upper="1e10" effort="27" velocity="26"/>
+                        origin_xyz="0.14 0 -0.025" origin_rpy="0 0 0.13433" axis_xyz="0 0 1" lower="-1e10" upper="1e10" effort="27" velocity="26"/>
 </robot>

Commit message: Add vmc into asm.

File: urdf/diablo_ASM.urdf (robot description, URDF)
Before this commit: robot diablo_ASM, 7 links, 6 joints
Joints:
- joint left_wheel_joint: limit effort=27 velocity=26 -> effort=5 velocity=26
- joint right_wheel_joint: limit effort=27 velocity=26 -> effort=5 velocity=26
